Commit message: working towards urdf

File: urdf/sevenDOF.urdf (robot description, URDF)
Before this commit: robot sevenDOF, 36 links, 35 joints
Links:
- link mount1: geometry collision cylinder length=0.2 radius=0.02; visual mesh filename=package://hw7code/meshes/Slider_Shaft.stl

File: urdf/stewart.urdf (robot description, URDF)
Before this commit: robot threeDOF, 2 links, 1 joints
Links:
- added link link1
- added link link2
- added link link3
- added link slider-base; visual mesh filename=package://finalprojectcode/meshes/Slider_Base.dae
- added link slider-shaft; visual mesh filename=package://finalprojectcode/meshes/Slider_Shaft.dae
- added link top; visual mesh filename=package://finalprojectcode/meshes/Platform_Top.dae
- added link uj-shaft; visual mesh filename=package://finalprojectcode/meshes/UJ_Shaft.dae
Joints:
- added joint attach-joint1: type fixed, parent link1, child uj-shaft
- added joint attach-joint2: type fixed, parent link2, child slider-base
- added joint attach-joint3: type fixed, parent link3, child slider-shaft
- added joint attach-top: type fixed, parent world, child top
- added joint d3: type prismatic, parent link2, child link3, origin xyz=0 0 -0.4 rpy=0 0 0, axis 0 0 -1, limit lower=0 upper=1.5 effort=1000.0 velocity=0.5
- added joint shifttotip: type fixed, parent link3, child tip, origin xyz=0 0 0 rpy=0 0 0
- added joint theta2: type continuous, parent link1, child link2, origin xyz=0 0 0 rpy=0 0 0, axis 0 1 0
- joint theta1: axis 0 0 1 -> 1 0 0; child tip -> link1; limit lower=-2.5 upper=2.5 effort=1000.0 velocity=0.5 -> (none); origin xyz=0 0 0 rpy=0 0 0 -> xyz=0 1.25 -0.2 rpy=0 0 0; type prismatic -> continuous

File: urdf/threeDOF.urdf (robot description, URDF)
Before this commit: robot threeDOF, 16 links, 15 joints
Links:
- link table: geometry visual mesh filename=package://finalprojectcode/meshes/Platform_Top.dae
