Commit message: 7 december updates

File: urdf/temp.urdf (robot description, URDF)
Before this commit: robot stewart, 31 links, 30 joints
Links:
- removed link leg1-platform
- removed link leg2-platform
- removed link leg3-platform
- removed link leg4-platform
- removed link leg5-platform
- removed link leg6-platform
- link leg1-uj-shaft: geometry visual mesh filename=package://finalprojectcode/meshes/UJ_Shaft.dae
- link world: geometry visual mesh filename=package://finalprojectcode/meshes/Platform_Top.dae
Joints:
- removed joint leg1-tip-to-platform
- removed joint leg2-tip-to-platform
- removed joint leg3-tip-to-platform
- removed joint leg4-tip-to-platform
- removed joint leg5-tip-to-platform
- removed joint leg6-tip-to-platform
- joint leg1-pitch: origin xyz=0 1.25 0.2 rpy=0 0 0 -> xyz=0 1.25 -0.2 rpy=0 0 0
- joint leg1-prismatic: origin xyz=0 0 0.4 rpy=3.14159 0 0 -> xyz=0 0 -0.4 rpy=0 0 0
- joint leg1-to-tip: origin xyz=0 0 -1.5 rpy=0 0 0 -> xyz=0 0 0 rpy=0 0 0
- joint leg2-pitch: origin xyz=-1.08253 0.625 0.2 rpy=0 0 1.04719 -> xyz=-1.08253 0.625 -0.2 rpy=0 0 1.04719
- joint leg2-prismatic: origin xyz=0 0 0.4 rpy=3.14159 0 0 -> xyz=0 0 -0.4 rpy=0 0 0
- joint leg2-to-tip: origin xyz=0 0 -1.5 rpy=0 0 0 -> xyz=0 0 0 rpy=0 0 0
- joint leg3-pitch: origin xyz=-1.08253 -0.625 0.2 rpy=0 0 2.094395 -> xyz=-1.08253 -0.625 -0.2 rpy=0 0 2.094395
- joint leg3-prismatic: origin xyz=0 0 0.4 rpy=3.14159 0 0 -> xyz=0 0 -0.4 rpy=0 0 0
- joint leg3-to-tip: origin xyz=0 0 -1.5 rpy=0 0 0 -> xyz=0 0 0 rpy=0 0 0
- joint leg4-pitch: origin xyz=0 -1.25 0.2 rpy=0 0 0 -> xyz=0 -1.25 -0.2 rpy=0 0 0
- joint leg4-prismatic: origin xyz=0 0 0.4 rpy=3.14159 0 0 -> xyz=0 0 -0.4 rpy=0 0 0
- joint leg4-to-tip: origin xyz=0 0 -1.5 rpy=0 0 0 -> xyz=0 0 0 rpy=0 0 0
- joint leg5-pitch: origin xyz=1.0825317 -0.625 0.2 rpy=0 0 1.047197 -> xyz=1.0825317 -0.625 -0.2 rpy=0 0 1.047197
- joint leg5-prismatic: origin xyz=0 0 0.4 rpy=3.14159 0 0 -> xyz=0 0 -0.4 rpy=0 0 0
- joint leg5-to-tip: origin xyz=0 0 -1.5 rpy=0 0 0 -> xyz=0 0 0 rpy=0 0 0
- joint leg6-pitch: origin xyz=1.0825317 0.625 0.2 rpy=0 0 -1.047197 -> xyz=1.0825317 0.625 -0.2 rpy=0 0 -1.047197
- joint leg6-prismatic: origin xyz=0 0 0.4 rpy=3.14159 0 0 -> xyz=0 0 -0.4 rpy=0 0 0
- joint leg6-to-tip: origin xyz=0 0 -1.5 rpy=0 0 0 -> xyz=0 0 0 rpy=0 0 0
