Commit message: updated stewart

File: urdf/stewart.urdf (robot description, URDF)
Before this commit: robot stewart, 9 links, 8 joints
Links:
- removed link link1
- removed link link2
- removed link link3
- removed link slider-base
- removed link slider-shaft
- removed link tip
- removed link top
- removed link uj-shaft
- added link leg1-slider-base; visual mesh filename=package://finalprojectcode/meshes/Slider_Base.dae
- added link leg1-slider-shaft; visual mesh filename=package://finalprojectcode/meshes/Slider_Shaft.dae
- added link leg1-tip
- added link leg1-uj-shaft; visual mesh filename=package://finalprojectcode/meshes/UJ_Shaft.dae
- added link leg2-slider-base; visual mesh filename=package://finalprojectcode/meshes/Slider_Base.dae
- added link leg2-slider-shaft; visual mesh filename=package://finalprojectcode/meshes/Slider_Shaft.dae
- added link leg2-tip
- added link leg2-uj-shaft; visual mesh filename=package://finalprojectcode/meshes/UJ_Shaft.dae
- added link leg3-slider-base; visual mesh filename=package://finalprojectcode/meshes/Slider_Base.dae
- added link leg3-slider-shaft; visual mesh filename=package://finalprojectcode/meshes/Slider_Shaft.dae
- added link leg3-tip
- added link leg3-uj-shaft; visual mesh filename=package://finalprojectcode/meshes/UJ_Shaft.dae
- added link leg4-slider-base; visual mesh filename=package://finalprojectcode/meshes/Slider_Base.dae
- added link leg4-slider-shaft; visual mesh filename=package://finalprojectcode/meshes/Slider_Shaft.dae
- added link leg4-tip
- added link leg4-uj-shaft; visual mesh filename=package://finalprojectcode/meshes/UJ_Shaft.dae
- added link leg5-slider-base; visual mesh filename=package://finalprojectcode/meshes/Slider_Base.dae
- added link leg5-slider-shaft; visual mesh filename=package://finalprojectcode/meshes/Slider_Shaft.dae
- added link leg5-tip
- added link leg5-uj-shaft; visual mesh filename=package://finalprojectcode/meshes/UJ_Shaft.dae
- added link leg6-slider-base; visual mesh filename=package://finalprojectcode/meshes/Slider_Base.dae
- added link leg6-slider-shaft; visual mesh filename=package://finalprojectcode/meshes/Slider_Shaft.dae
- added link leg6-tip
- added link leg6-uj-shaft; visual mesh filename=package://finalprojectcode/meshes/UJ_Shaft.dae
- link world: geometry visual mesh filename=package://finalprojectcode/meshes/Platform_Top.dae
Joints:
- removed joint attach-joint1
- removed joint attach-joint2
- removed joint attach-joint3
- removed joint attach-top
- removed joint d3
- removed joint shifttotip
- removed joint theta1
- removed joint theta2
- added joint leg1-pitch: type continuous, parent world, child leg1-uj-shaft, origin xyz=0 1.25 -0.2 rpy=0 0 0, axis 1 0 0
- added joint leg1-prismatic: type prismatic, parent leg1-slider-base, child leg1-slider-shaft, origin xyz=0 0 -0.4 rpy=0 0 0, axis 0 0 -1, limit lower=0 upper=1.5 effort=1000.0 velocity=0.5
- added joint leg1-roll: type continuous, parent leg1-uj-shaft, child leg1-slider-base, origin xyz=0 0 0 rpy=0 0 0, axis 0 1 0
- added joint leg1-to-tip: type fixed, parent leg1-slider-shaft, child leg1-tip, origin xyz=0 0 0 rpy=0 0 0
- added joint leg2-pitch: type continuous, parent world, child leg2-uj-shaft, origin xyz=-1.08253 0.625 -0.2 rpy=0 0 1.04719, axis 1 0 0
- added joint leg2-prismatic: type prismatic, parent leg2-slider-base, child leg2-slider-shaft, origin xyz=0 0 -0.4 rpy=0 0 0, axis 0 0 -1, limit lower=0 upper=1.5 effort=1000.0 velocity=0.5
- added joint leg2-roll: type continuous, parent leg2-uj-shaft, child leg2-slider-base, origin xyz=0 0 0 rpy=0 0 0, axis 0 1 0
- added joint leg2-to-tip: type fixed, parent leg2-slider-shaft, child leg2-tip, origin xyz=0 0 0 rpy=0 0 0
- added joint leg3-pitch: type continuous, parent world, child leg3-uj-shaft, origin xyz=-1.08253 -0.625 -0.2 rpy=0 0 2.094395, axis 1 0 0
- added joint leg3-prismatic: type prismatic, parent leg3-slider-base, child leg3-slider-shaft, origin xyz=0 0 -0.4 rpy=0 0 0, axis 0 0 -1, limit lower=0 upper=1.5 effort=1000.0 velocity=0.5
- added joint leg3-roll: type continuous, parent leg3-uj-shaft, child leg3-slider-base, origin xyz=0 0 0 rpy=0 0 0, axis 0 1 0
- added joint leg3-to-tip: type fixed, parent leg3-slider-shaft, child leg3-tip, origin xyz=0 0 0 rpy=0 0 0
- added joint leg4-pitch: type continuous, parent world, child leg4-uj-shaft, origin xyz=0 -1.25 -0.2 rpy=0 0 0, axis 1 0 0
- added joint leg4-prismatic: type prismatic, parent leg4-slider-base, child leg4-slider-shaft, origin xyz=0 0 -0.4 rpy=0 0 0, axis 0 0 -1, limit lower=0 upper=1.5 effort=1000.0 velocity=0.5
- added joint leg4-roll: type continuous, parent leg4-uj-shaft, child leg4-slider-base, origin xyz=0 0 0 rpy=0 0 0, axis 0 1 0
- added joint leg4-to-tip: type fixed, parent leg4-slider-shaft, child leg4-tip, origin xyz=0 0 0 rpy=0 0 0
- added joint leg5-pitch: type continuous, parent world, child leg5-uj-shaft, origin xyz=1.0825317 -0.625 -0.2 rpy=0 0 1.047197, axis 1 0 0
- added joint leg5-prismatic: type prismatic, parent leg5-slider-base, child leg5-slider-shaft, origin xyz=0 0 -0.4 rpy=0 0 0, axis 0 0 -1, limit lower=0 upper=1.5 effort=1000.0 velocity=0.5
- added joint leg5-roll: type continuous, parent leg5-uj-shaft, child leg5-slider-base, origin xyz=0 0 0 rpy=0 0 0, axis 0 1 0
- added joint leg5-to-tip: type fixed, parent leg5-slider-shaft, child leg5-tip, origin xyz=0 0 0 rpy=0 0 0
- added joint leg6-pitch: type continuous, parent world, child leg6-uj-shaft, origin xyz=1.0825317 0.625 -0.2 rpy=0 0 -1.047197, axis 1 0 0
- added joint leg6-prismatic: type prismatic, parent leg6-slider-base, child leg6-slider-shaft, origin xyz=0 0 -0.4 rpy=0 0 0, axis 0 0 -1, limit lower=0 upper=1.5 effort=1000.0 velocity=0.5
- added joint leg6-roll: type continuous, parent leg6-uj-shaft, child leg6-slider-base, origin xyz=0 0 0 rpy=0 0 0, axis 0 1 0
- added joint leg6-to-tip: type fixed, parent leg6-slider-shaft, child leg6-tip, origin xyz=0 0 0 rpy=0 0 0

Commit message: platform top

File: urdf/stewart.urdf (robot description, URDF)
Before this commit: robot stewart, 31 links, 30 joints
Links:
- link leg1-uj-shaft: geometry visual mesh filename=package://finalprojectcode/meshes/UJ_Shaft.dae
- link leg6-platform: geometry visual mesh filename=package://finalprojectcode/meshes/Platform_Top.dae
Joints:
- joint leg1-pitch: origin xyz=0 1.25 0.2 rpy=0 0 0 -> xyz=0.25 1.5 0.3 rpy=0 0 0
- joint leg2-pitch: origin xyz=-1.08253 0.625 0.2 rpy=0 0 1.04719 -> xyz=-0.25 1.50 0.3 rpy=0 0 0
- joint leg3-pitch: origin xyz=-1.08253 -0.625 0.2 rpy=0 0 2.094395 -> xyz=-1.424038 -0.533494 0.3 rpy=0 0 2.094395
- joint leg4-pitch: origin xyz=0 -1.25 0.2 rpy=0 0 0 -> xyz=-1.1174038 -0.96650635 0.3 rpy=0 0 2.094395
- joint leg5-pitch: origin xyz=1.0825317 -0.625 0.2 rpy=0 0 1.047197 -> xyz=1.1174038 -0.966506 0.3 rpy=0 0 0
- joint leg6-pitch: origin xyz=1.0825317 0.625 0.2 rpy=0 0 -1.047197 -> xyz=1.424038 -0.533494 0.3 rpy=0 0 1.047197
- joint leg6-tip-to-platform: origin xyz=0 1.25 -0.2 rpy=0 0 0 -> xyz=0 0 -0.2 rpy=0 0 0

Commit message: trajectory demos

File: urdf/stewart.urdf (robot description, URDF)
Before this commit: robot stewart, 31 links, 30 joints
Links:
- removed link leg1-platform
- removed link leg2-platform
- removed link leg3-platform
- removed link leg4-platform
- removed link leg5-platform
- removed link leg6-platform
Joints:
- removed joint leg1-tip-to-platform
- removed joint leg2-tip-to-platform
- removed joint leg3-tip-to-platform
- removed joint leg4-tip-to-platform
- removed joint leg5-tip-to-platform
- removed joint leg6-tip-to-platform
- joint leg1-pitch: axis 1 0 0 -> 0 1 0
- joint leg1-prismatic: limit lower=0 upper=1.5 effort=1000.0 velocity=0.5 -> lower=0 upper=1.8 effort=1000.0 velocity=0.5
- joint leg1-roll: axis 0 1 0 -> 1 0 0
- joint leg2-pitch: axis 1 0 0 -> 0 1 0
- joint leg2-prismatic: limit lower=0 upper=1.5 effort=1000.0 velocity=0.5 -> lower=0 upper=1.8 effort=1000.0 velocity=0.5
- joint leg2-roll: axis 0 1 0 -> 1 0 0
- joint leg3-pitch: axis 1 0 0 -> 0 1 0; origin xyz=-1.424038 -0.533494 0.3 rpy=0 0 2.094395 -> xyz=-1.424038 -0.533494 0.3 rpy=0 0 0
- joint leg3-prismatic: limit lower=0 upper=1.5 effort=1000.0 velocity=0.5 -> lower=0 upper=1.8 effort=1000.0 velocity=0.5
- joint leg3-roll: axis 0 1 0 -> 1 0 0
- joint leg4-pitch: axis 1 0 0 -> 0 1 0; origin xyz=-1.1174038 -0.96650635 0.3 rpy=0 0 2.094395 -> xyz=-1.1174038 -0.96650635 0.3 rpy=0 0 0
- joint leg4-prismatic: limit lower=0 upper=1.5 effort=1000.0 velocity=0.5 -> lower=0 upper=1.8 effort=1000.0 velocity=0.5
- joint leg4-roll: axis 0 1 0 -> 1 0 0
- joint leg5-pitch: axis 1 0 0 -> 0 1 0
- joint leg5-prismatic: limit lower=0 upper=1.5 effort=1000.0 velocity=0.5 -> lower=0 upper=1.8 effort=1000.0 velocity=0.5
- joint leg5-roll: axis 0 1 0 -> 1 0 0
- joint leg6-pitch: axis 1 0 0 -> 0 1 0; origin xyz=1.424038 -0.533494 0.3 rpy=0 0 1.047197 -> xyz=1.424038 -0.533494 0.3 rpy=0 0 0
- joint leg6-prismatic: limit lower=0 upper=1.5 effort=1000.0 velocity=0.5 -> lower=0 upper=1.8 effort=1000.0 velocity=0.5
- joint leg6-roll: axis 0 1 0 -> 1 0 0
